Commit message: Messy overhaul

File: urdf/gtr2.urdf.xacro (robot description, xacro)
@@ -9,5 +9,5 @@
   <xacro:include filename="$(find gait_training_robot)/urdf/azure_kinect.urdf.xacro" />
   <xacro:azure_kinect_xacro name="rear_kinect" parent="camera_mount_top">
-	  <origin rpy="0 0 3.1416" xyz="-0.07 0 0.01"/>
+	  <origin rpy="0 -0.0225 3.1416" xyz="-0.07 0 0.01"/>
   </xacro:azure_kinect_xacro>
 	<!-- kinect v1 description -->

Commit message: Fix static transform from robot to kinect

File: urdf/gtr2.urdf.xacro (robot description, xacro)
@@ -9,5 +9,5 @@
   <xacro:include filename="$(find gait_training_robot)/urdf/azure_kinect.urdf.xacro" />
   <xacro:azure_kinect_xacro name="rear_kinect" parent="camera_mount_top">
-	  <origin rpy="0 -0.0225 3.1416" xyz="-0.07 0 0.01"/>
+	  <origin rpy="0 -0.0225 3.1416" xyz="-0.028 0.023 0.01"/>
   </xacro:azure_kinect_xacro>
 	<!-- kinect v1 description -->
