Commit message: fix urdf path error

File: urdf/kinect.urdf.xacro (robot description, xacro)
@@ -15,5 +15,5 @@
         <origin xyz="-0.05 -0.17 -0.02" rpy="${M_PI/2.0} 0 ${M_PI/2.0}"/>
         <geometry>
-          <mesh filename="package://amr_robots_description/meshes/gtr/68-04546_Kinect_Sensor--coarse.STL" scale="0.001 0.001 0.001" />
+          <mesh filename="package://gait_training_robot/meshes/68-04546_Kinect_Sensor--coarse.STL" scale="0.001 0.001 0.001" />
         </geometry>
         <material name="gray">

Commit message: update xacro tag name

File: urdf/kinect.urdf.xacro (robot description, xacro)
@@ -2,5 +2,5 @@
 <robot name="kinect" xmlns:xacro="http://ros.org/wiki/xacro">
   <xacro:macro name="kinect_xacro" params="name parent *origin">
-    <property name="M_PI" value="3.14159"/>
+    <xacro:property name="M_PI" value="3.14159"/>
     <joint name="${name}_joint" type="fixed">
       <xacro:insert_block name="origin"/>
